Commit message: Update xacro files to include stl files, and fix minor issue at example.launch.py

File: velodyne_description/urdf/HDL-32E.urdf.xacro (robot description, xacro)
@@ -18,5 +18,6 @@
       <visual>
         <geometry>
-          <mesh filename="package://velodyne_description/meshes/HDL32E_base.dae" />
+          <!-- <mesh filename="package://velodyne_description/meshes/HDL32E_base.dae" /> -->
+          <mesh filename="file://$(find velodyne_description)/meshes/HDL32E_base.dae" />
         </geometry>
       </visual>
@@ -42,5 +43,6 @@
         <origin xyz="0 0 -0.09081" rpy="0 0 0" />
         <geometry>
-          <mesh filename="package://velodyne_description/meshes/HDL32E_scan.dae" />
+          <!-- <mesh filename="package://velodyne_description/meshes/HDL32E_scan.dae" /> -->
+          <mesh filename="file://$(find velodyne_description)/meshes/HDL32E_scan.dae" />
         </geometry>
       </visual>

File: velodyne_description/urdf/VLP-16.urdf.xacro (robot description, xacro)
@@ -18,10 +18,12 @@
       <visual>
         <geometry>
-          <mesh filename="package://velodyne_description/meshes/VLP16_base_1.dae" />
+          <!-- <mesh filename="package://velodyne_description/meshes/VLP16_base_1.dae" /> -->
+          <mesh filename="file://$(find velodyne_description)/meshes/VLP16_base_1.dae" />
         </geometry>
       </visual>
       <visual>
         <geometry>
-          <mesh filename="package://velodyne_description/meshes/VLP16_base_2.dae" />
+          <!-- <mesh filename="package://velodyne_description/meshes/VLP16_base_2.dae" /> -->
+          <mesh filename="file://$(find velodyne_description)/meshes/VLP16_base_2.dae" />
         </geometry>
       </visual>
@@ -47,5 +49,6 @@
         <origin xyz="0 0 -0.0377" />
         <geometry>
-          <mesh filename="package://velodyne_description/meshes/VLP16_scan.dae" />
+          <!-- <mesh filename="package://velodyne_description/meshes/VLP16_scan.dae" /> -->
+          <mesh filename="file://$(find velodyne_description)/meshes/VLP16_scan.dae" />
         </geometry>
       </visual>
